File: HDK/SCKB-Xin.kicad_sch (KiCad schematic)
At the start: 127 parts, among them SW1 SW_Push, SW10 SW_Push, SW11 SW_Push, SW12 SW_Push, SW13 SW_Push, SW14 SW_Push, SW15 SW_Push, SW16 SW_Push, SW17 SW_Push, SW18 SW_Push, SW19 SW_Push, SW2 SW_Push, SW20 SW_Push, SW21 SW_Push, SW22 SW_Push, SW23 SW_Push, SW24 SW_Push, SW25 SW_Push, SW26 SW_Push, SW27 SW_Push, SW28 SW_Push, SW29 SW_Push, SW3 SW_Push, SW30 SW_Push, SW31 SW_Push, SW32 SW_Push, SW33 SW_Push, SW34 SW_Push, SW35 SW_Push, SW36 SW_Push, SW37 SW_Push, SW38 SW_Push, SW39 SW_Push, SW4 SW_Push, SW40 SW_Push, SW41 SW_Push, SW42 SW_Push, SW43 SW_Push, SW44 SW_Push, SW45 SW_Push, SW46 SW_Push, SW47 SW_Push, SW48 SW_Push, SW49 SW_Push, SW5 SW_Push, SW50 SW_Push, SW51 SW_Push, SW52 SW_Push, SW53 SW_Push, SW54 SW_Push, SW55 SW_Push, SW56 SW_Push, SW57 SW_Push, SW58 SW_Push, SW59 SW_Push, SW6 SW_Push, SW60 SW_Push, SW61 SW_Push, SW62 SW_Push, SW63 SW_Push, SW64 SW_Push, SW65 SW_Push, SW66 SW_Push, SW67 SW_Push, SW68 SW_Push, SW69 SW_Push, SW7 SW_Push, SW70 SW_Push, SW71 SW_Push, SW72 SW_Push, SW73 SW_Push, SW74 SW_Push, SW75 SW_Push, SW76 SW_Push, SW77 SW_Push, SW78 SW_Push, SW79 SW_Push, SW8 SW_Push, SW80 SW_Push, SW81 SW_Push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

Commit message: updated
Parts:
- removed D1, D10, D11, D12, D13, D14, D15, D16, D17, D18, D19, D2, D20, D21, D22, D23, D24, D25, D26, D27, D28, D29, D3, D30, D31, D32, D33, D34, D35, D36, D37, D38, D39, D4, D40, D41, D42, D43, D5, D6, D7, D8, D9: D, Package_TO_SOT_SMD:SOT-23, symbol SCKB-Kicad-Rsc:CC-D
- removed SW1, SW10, SW11, SW12, SW13, SW14, SW15, SW16, SW17, SW18, SW19, SW2, SW20, SW21, SW22, SW23, SW24, SW25, SW26, SW27, SW28, SW29, SW3, SW30, SW31, SW32, SW33, SW34, SW35, SW36, SW37, SW38, SW39, SW4, SW40, SW41, SW42, SW43, SW44, SW45, SW46, SW47, SW48, SW49, SW5, SW50, SW51, SW52, SW53, SW54, SW55, SW56, SW57, SW58, SW59, SW6, SW60, SW61, SW62, SW63, SW64, SW65, SW66, SW67, SW68, SW69, SW7, SW70, SW71, SW72, SW73, SW74, SW75, SW76, SW77, SW78, SW79, SW8, SW80, SW81, SW82, SW83, SW9: SW_Push, PCM_Switch_Keyboard_Cherry_MX:SW_Cherry_MX_PCB_1.00u, symbol Switch:SW_Push
- removed U1: STM32F072RBTx, Package_QFP:LQFP-64_10x10mm_P0.5mm, symbol MCU_ST_STM32F0:STM32F072RBTx
- added C101, C102, C103, C104, C105, C108, C109, C112, C113: 100n, lib:C_0402_1005Metric, symbol Device:C
- added C106: 4u7, lib:C_0603_1608Metric, symbol Device:C
- added C107, C110, C111: 10u, lib:C_0603_1608Metric, symbol Device:C
- added C114, C115: 30p, lib:C_0603_1608Metric, symbol Device:C
- added D101, D102: CESD5V0D3, lib:D_SOD-323, symbol Device:D_Zener
- added D103, D104: LED, symbol Device:LED
- added J101: Conn_01x04, symbol Connector_Generic:Conn_01x04
- added L101: CBG160808U121T, lib:L_0603_1608Metric, symbol Device:L_Ferrite
- added R101, R102: 10k, lib:R_0402_1005Metric, symbol Device:R
- added R103, R104: 3k, lib:R_0402_1005Metric, symbol Device:R
- added SW101: NRST, symbol Switch:SW_Push
- added SW102: BOOT0, symbol Switch:SW_Push
- added U101: AMS1117-3.3, lib:SOT-223-3_TabPin2, symbol Regulator_Linear:AMS1117-3.3
- added U102: STM32F103RBTx, lib:LQFP-64_10x10mm_P0.5mm, symbol MCU_ST_STM32F1:STM32F103RBTx
- added Y101: 8Mhz, lib:Crystal_SMD_5032-2Pin_5.0x3.2mm, symbol Device:Crystal
Connections:
- net C10: now also U102.57 (PB5)
- net C11: now also U102.51 (PC10)
- net C12: now also U102.52 (PC11)
- net C13: now also U102.53 (PC12)
- new net: D103.1 (K), R103.1
- new net: D104.1 (K), R104.1
- new net +3V3: C101.1, C102.1, C103.1, C104.1, C105.1, C106.1, C111.1, C112.1, D102.1 (K), D103.2 (A), D104.2 (A), L101.1, R101.1, SW102.1, U101.2 (VO), U102.1 (VBAT), U102.19 (VDD), U102.32 (VDD), U102.48 (VDD), U102.64 (VDD)
- new net +3V3A: C107.1, C108.1, L101.2, U102.13 (VDDA)
- new net BOOT0: R102.1, SW102.2, U102.60 (BOOT0)
- new net C01: U102.2 (PC13)
- new net C02: U102.3 (PC14)
- new net C03: U102.4 (PC15)
- new net C04: U102.16 (PA2)
- new net C05: U102.17 (PA3)
- new net C06: U102.33 (PB12)
- new net C07: U102.50 (PA15)
- new net C08: U102.34 (PB13)
- new net C09: U102.35 (PB14)
- new net C14: U102.54 (PD2)
- new net C15: U102.55 (PB3)
- new net C16: U102.56 (PB4)
- new net GND: C101.2, C102.2, C103.2, C104.2, C105.2, C106.2, C107.2, C108.2, C109.2, C110.2, C111.2, C112.2, C113.2, C114.1, C115.1, D101.2 (A), D102.2 (A), J101.4 (Pin_4), R102.2, R103.2, R104.2, SW101.1, U101.1 (GND), U102.12 (VSSA), U102.18 (VSS), U102.31 (VSS), U102.47 (VSS), U102.63 (VSS)
- new net HSE_IN: C114.2, U102.5 (PD0), Y101.1
- new net HSE_OUT: C115.2, U102.6 (PD1), Y101.2
- new net NRST: C113.1, R101.2, SW101.2, U102.7 (NRST)
- new net R01: U102.21 (PA5)
- new net R02: U102.22 (PA6)
- new net R03: U102.23 (PA7)
- new net R04: U102.41 (PA8)
- new net R05: U102.42 (PA9)
- new net R06: U102.62 (PB9)
- new net SWCLK: U102.49 (PA14)
- new net SWDIO: U102.46 (PA13)
- new net USB_D+: J101.3 (Pin_3), U102.45 (PA12)
- new net USB_D-: J101.2 (Pin_2), U102.44 (PA11)
- new net VBUS: C109.1, C110.1, D101.1 (K), J101.1 (Pin_1), U101.3 (VI)
- no-connect marks 3 -> 0
Other:
- added sheet KeyMatrix (KeyMatrix.kicad_sch)
